File: Lab/Assignment1/Lab_assignment1.kicad_sch (KiCad schematic)
At the start: 30 parts, among them P1 Conn_02x03_Odd_Even, P2 SWD, P3 Conn_01x20, P4 Conn_01x20, SW1 SW_Push, U1 STM32F103C8Tx, U2 AMS1117-3.3, U3 USB_B_Micro, Y2 8MHZ

Commit message: UPD  Solving
Solving the first assignment for the Embedded Systems Lab
Connections:
- net 5V renamed VCC
